Commit message: dieu khien xe

File: install/car_3_wheel/share/car_3_wheel/urdf/ver6.urdf (robot description, URDF)
Before this commit: robot ver4, 6 links, 5 joints
Links:
- link base_link: mass 12.8783005904919 -> 0.12
- link car_left: mass 0.579007065567467 -> 0.1403
- link car_right: mass 0.579007235319938 -> 0.1403
- link caster: mass 0.0206098306469479 -> 0.5
Joints:
- joint caster_joint: origin xyz=0.093013 0.012666 0.0995 rpy=0 0 0 -> xyz=0.093013 0.012666 0.0995 rpy=0 0 -3.1408
- joint caster_wheel_joint: axis 0.76732 0 -0.64126 -> 0 0 1

File: src/car_3_wheel/urdf/ver6.urdf (robot description, URDF)
Before this commit: robot ver4, 6 links, 5 joints
Links:
- link base_link: mass 12.8783005904919 -> 0.12
- link car_left: mass 0.579007065567467 -> 0.1403
- link car_right: mass 0.579007235319938 -> 0.1403
- link caster: mass 0.0206098306469479 -> 0.5

Commit message: map+xe

File: install/car_3_wheel/share/car_3_wheel/urdf/ver6.urdf (robot description, URDF)
Before this commit: robot ver6, 6 links, 5 joints
Joints:
- joint caster_joint: origin xyz=0.093013 0.012666 0.0995 rpy=0 0 -3.1408 -> xyz=0.093013 0.012666 0.0995 rpy=0 0 0
- joint caster_wheel_joint: axis 0 0 1 -> 0.76732 0 -0.64126
